File: raven-main/Detector-Power-Board/_restore_backup_2026-08-23T18-58-27-726/detector-power.kicad_sch (KiCad schematic)
At the start: 35 parts, among them J1 DeployLipo, J2 Conn_01x04, J9 UCLipo, U1 LT8330IS6-TRMPBF, U2 TPS22810DRV, U3 LM317LCLPRE3, U4 LM317LCLPRE3

Commit message: Replaced LDO with correct one
Parts:
- removed U4: LM317LCLPRE3, LM317MDT_TR:DPAK_STM, symbol LM317MDT_TR:LM317MDT-TR
- added CR1: LM317MDT-TR, DPAK_STM, symbol LM317MDT_TR:LM317MDT-TR
- U3: footprint LM317MDT_TR:DPAK_STM -> DPAK_STM
Connections:
- net Filtered_Power_Out_25V: no longer C8.2, D6.1 (K), R6.1
- net Power_Out_27.5V: now also CR1.2 (VIN)
- net at C10.2, D6.2 (A), R5.1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: now also CR1.1 (ADJUST)
- net at C9.2, D3.2 (A), R3.1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: no longer U3.1 (ADJUST)
- new net: C8.2, CR1.3 (VOUT), D6.1 (K), R6.1
Other:
- moved on the sheet: D4, U3
Changed lines of the file:
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@@
 	)
 	(junction
-		(at 97.79 99.06)
-		(diameter 0)
-		(color 0 0 0 0)
-	)
-	(junction
 		(at 210.82 87.63)
 		(diameter 0)
@@
 	)
 	(junction
-		(at 186.69 87.63)
+		(at 186.69 78.74)
 		(diameter 0)
 		(color 0 0 0 0)
@@
 	)
 	(junction
+		(at 97.79 99.06)
+		(diameter 0)
+		(color 0 0 0 0)
+	)
+	(junction
 		(at 118.11 170.18)
 		(diameter 0)
@@
 	)
 	(junction
-		(at 210.82 78.74)
-		(diameter 0)
-		(color 0 0 0 0)
-	)
-	(junction
 		(at 156.21 64.77)
 		(diameter 0)
@@
 	)
 	(junction
-		(at 116.84 99.06)
-		(diameter 0)
-		(color 0 0 0 0)
-	)
-	(junction
 		(at 55.88 167.64)
 		(diameter 0)
@@
 	(wire
 		(pts
-			(xy 210.82 78.74) (xy 165.1 78.74)
-		)
-		(stroke
-			(width 0)
-			(type default)
-		)
-	)
-	(wire
-		(pts
 			(xy 144.78 64.77) (xy 156.21 64.77)
 		)
@@
 	(wire
 		(pts
-			(xy 165.1 78.74) (xy 165.1 67.31)
-		)
-		(stroke
-			(width 0)
-			(type default)
-		)
-	)
-	(wire
-		(pts
 			(xy 48.26 31.75) (xy 53.34 31.75)
 		)
@@
 	(wire
 		(pts
-			(xy 186.69 87.63) (xy 193.04 87.63)
+			(xy 186.69 78.74) (xy 193.04 78.74)
 		)
 		(stroke
@@
 	(wire
 		(pts
+			(xy 200.66 87.63) (xy 200.66 78.74)
+		)
+		(stroke
+			(width 0)
+			(type default)
+		)
+	)
+	(wire
+		(pts
 			(xy 118.11 162.56) (xy 118.11 146.05)
 		)
@@
 	(wire
 		(pts
-			(xy 156.21 74.93) (xy 156.21 87.63)
+			(xy 156.21 74.93) (xy 156.21 78.74)
 		)
 		(stroke
@@
 	(wire
 		(pts
-			(xy 116.84 99.06) (xy 123.19 99.06)
-		)
-		(stroke
-			(width 0)
-			(type default)
-		)
-	)
-	(wire
-		(pts
 			(xy 52.07 110.49) (xy 86.36 110.49)
 		)
@@
 	(wire
 		(pts
-			(xy 186.69 87.63) (xy 186.69 90.17)
+			(xy 186.69 78.74) (xy 186.69 81.28)
 		)
 		(stroke
@@
 	(wire
 		(pts
-			(xy 156.21 87.63) (xy 186.69 87.63)
+			(xy 156.21 78.74) (xy 186.69 78.74)
 		)
 		(stroke
@@
 	)
 	(label "Filtered_Power_Out_25V"
-		(at 123.19 99.06 0)
+		(at 139.7 96.52 0)
 		(effects
 			(font
@@
 	(symbol
 		(lib_id "power:GND")
-		(at 186.69 90.17 0)
+		(at 186.69 81.28 0)
 		(unit 1)
 		(body_style 1)
@@
 		(fields_autoplaced yes)
 		(property "Reference" "#PWR012"
-			(at 186.69 96.52 0)
+			(at 186.69 87.63 0)
 			(hide yes)
 			(show_name no)
@@
 		)
 		(property "Value" "GND"
-			(at 186.69 95.25 0)
+			(at 186.69 86.36 0)
 			(show_name no)
 			(do_not_autoplace no)
@@
 		)
 		(property "Footprint" ""
-			(at 186.69 90.17 0)
+			(at 186.69 81.28 0)
 			(hide yes)
 			(show_name no)
@@
 		)
 		(property "Datasheet" ""
-			(at 186.69 90.17 0)
+			(at 186.69 81.28 0)
 			(hide yes)
 			(show_name no)
@@
 		)
 		(property "Description" "Power symbol creates a global label with name \"GND\" , ground"
-			(at 186.69 90.17 0)
+			(at 186.69 81.28 0)
 			(hide yes)
 			(show_name no)
@@
 	)
 	(symbol
-		(lib_id "LM317MDT_TR:LM317MDT-TR")
-		(at 52.07 101.6 0)
-		(mirror x)
-		(unit 1)
-		(body_style 1)
-		(exclude_from_sim no)
-		(in_bom yes)
-		(on_board yes)
-		(in_pos_files yes)
-		(dnp no)
-		(property "Reference" "U4"
-			(at 74.93 111.76 0)
-			(show_name no)
-			(do_not_autoplace no)
-			(effects
-				(font
-					(size 1.524 1.524)
-				)
-			)
-		)
-		(property "Value" "LM317LCLPRE3"
-			(at 74.93 109.22 0)
-			(show_name no)
-			(do_not_autoplace no)
-			(effects
-				(font
-					(size 1.524 1.524)
-				)
-			)
-		)
-		(property "Footprint" "LM317MDT_TR:DPAK_STM"
-			(at 52.07 101.6 0)
-			(hide yes)
-			(show_name no)
-			(do_not_autoplace no)
-			(effects
-				(font
-					(size 1.27 1.27)
-					(italic yes)
-				)
-			)
-		)
-		(property "Datasheet" "https://www.st.com/resource/en/datasheet/lm217m.pdf"
-			(at 52.07 101.6 0)
-			(hide yes)
-			(show_name no)
-			(do_not_autoplace no)
-			(effects
-				(font
-					(size 1.27 1.27)
-					(italic yes)
-				)
-			)
-		)
-		(property "Description" ""
-			(at 52.07 101.6 0)
-			(hide yes)
-			(show_name no)
-			(do_not_autoplace no)
-			(effects
-				(font
-					(size 1.27 1.27)
-				)
-			)
-		)
-		(pin "1"
-		)
-		(pin "3"
-		)
-		(pin "2"
-		)
-		(instances
-			(project "detector-power"
-				(path "/7c9dd221-ef7c-445c-ac49-d326ea2b82e0"
-					(reference "U4")
-					(unit 1)
-				)
-			)
-		)
-	)
-	(symbol
 		(lib_id "Device:D_Schottky")
 		(at 111.76 146.05 180)
@@
 	(symbol
 		(lib_id "Diode:1N4002")
-		(at 196.85 87.63 0)
+		(at 196.85 78.74 0)
 		(unit 1)
 		(body_style 1)
@@
 		(fields_autoplaced yes)
 		(property "Reference" "D4"
-			(at 196.85 81.6262 0)
+			(at 196.85 72.7362 0)
 			(show_name no)
 			(do_not_autoplace no)
@@
 		)
 		(property "Value" "1N4002"
-			(at 196.85 84.1662 0)
+			(at 196.85 75.2762 0)
 			(show_name no)
 			(do_not_autoplace no)
@@
 		)
 		(property "Footprint" "Diode_THT:D_DO-41_SOD81_P10.16mm_Horizontal"
-			(at 196.85 92.075 0)
+			(at 196.85 83.185 0)
 			(hide yes)
 			(show_name no)
@@
 		)
 		(property "Datasheet" "http://www.vishay.com/docs/88503/1n4001.pdf"
-			(at 196.85 87.63 0)
+			(at 196.85 78.74 0)
 			(hide yes)
 			(show_name no)
@@
 		)
 		(property "Description" "100V 1A General Purpose Rectifier Diode, DO-41"
-			(at 196.85 87.63 0)
+			(at 196.85 78.74 0)
 			(hide yes)
 			(show_name no)
@@
 		)
 		(property "Sim.Device" "D"
-			(at 196.85 87.63 0)
+			(at 196.85 78.74 0)
 			(hide yes)
 			(show_name no)
@@
 		)
 		(property "Sim.Pins" "1=K 2=A"
-			(at 196.85 87.63 0)
+			(at 196.85 78.74 0)
 			(hide yes)
 			(show_name no)
@@
 	(symbol
 		(lib_id "LM317MDT_TR:LM317MDT-TR")
-		(at 165.1 67.31 0)
-		(mirror x)
+		(at 165.1 62.23 0)
 		(unit 1)
 		(body_style 1)
@@
 		(in_pos_files yes)
 		(dnp no)
+		(fields_autoplaced yes)
 		(property "Reference" "U3"
-			(at 187.96 77.47 0)
+			(at 187.96 52.07 0)
 			(show_name no)
 			(do_not_autoplace no)
@@
 		)
 		(property "Value" "LM317LCLPRE3"
-			(at 187.96 74.93 0)
+			(at 187.96 54.61 0)
 			(show_name no)
 			(do_not_autoplace no)
@@
 			)
 		)
-		(property "Footprint" "LM317MDT_TR:DPAK_STM"
-			(at 165.1 67.31 0)
+		(property "Footprint" "DPAK_STM"
+			(at 165.1 62.23 0)
 			(hide yes)
 			(show_name no)
@@
 		)
 		(property "Datasheet" "https://www.st.com/resource/en/datasheet/lm217m.pdf"
-			(at 165.1 67.31 0)
+			(at 165.1 62.23 0)
 			(hide yes)
 			(show_name no)
@@
 		)
 		(property "Description" ""
-			(at 165.1 67.31 0)
+			(at 165.1 62.23 0)
 			(hide yes)
 			(show_name no)
@@
 					(unit 1)
 				)
+			)
+		)
+	)
+	(symbol
+		(lib_id "LM317MDT_TR:LM317MDT-TR")
+		(at 52.07 101.6 0)
+		(mirror x)
+		(unit 1)
+		(body_style 1)
+		(exclude_from_sim no)
+		(in_bom yes)
+		(on_board yes)
+		(in_pos_files yes)
+		(dnp no)
+		(property "Reference" "CR1"
+			(at 74.93 111.76 0)
+			(show_name no)
+			(do_not_autoplace no)
+			(effects
+				(font
+					(size 1.524 1.524)
+				)
+			)
+		)
+		(property "Value" "LM317MDT-TR"
+			(at 74.93 109.22 0)
+			(show_name no)
+			(do_not_autoplace no)
+			(effects
+				(font
+					(size 1.524 1.524)
+				)
+			)
+		)
+		(property "Footprint" "DPAK_STM"
+			(at 52.07 101.6 0)
+			(hide yes)
+			(show_name no)
+			(do_not_autoplace no)
+			(effects
+				(font
+					(size 1.27 1.27)
+					(italic yes)
+				)
+			)
+		)
+		(property "Datasheet" "https://www.st.com/resource/en/datasheet/lm217m.pdf"
+			(at 52.07 101.6 0)
+			(hide yes)
+			(show_name no)
+			(do_not_autoplace no)
+			(effects
+				(font
+					(size 1.27 1.27)
+					(italic yes)
+				)
+			)
+		)
+		(property "Description" ""
+			(at 52.07 101.6 0)
+			(hide yes)
+			(show_name no)
+			(do_not_autoplace no)
+			(effects
+				(font
+					(size 1.27 1.27)
+				)
+			)
+		)
+		(pin "1"
+		)
+		(pin "2"
+		)
+		(pin "3"
+		)
+		(instances
+			(project "detector-power"
+				(path "/7c9dd221-ef7c-445c-ac49-d326ea2b82e0"
+					(reference "CR1")
+					(unit 1)
+				)
