File: raven-main/Detector-Power-Board/detector-power.kicad_sch (KiCad schematic)
At the start: 35 parts, among them J1 DeployLipo, J2 Conn_01x04, J9 UCLipo, U1 LT8330IS6-TRMPBF, U2 TPS22810DRV, U3 LM317LCLPRE3, U4 LM317LCLPRE3

Commit message: power board done
Parts:
- removed C1, C5: 4.7u, Capacitor_SMD:C_0805_2012Metric, symbol Device:C
- removed C10, C2, C7, C8, C9: 1u, Capacitor_SMD:C_0805_2012Metric, symbol Device:C
- removed C11: 1n, Capacitor_SMD:C_0805_2012Metric, symbol Device:C
- removed C12: 5u, Capacitor_SMD:C_0805_2012Metric, symbol Device:C
- removed C13, C6: 0.1u, Capacitor_SMD:C_0805_2012Metric, symbol Device:C
- removed C3: 4.7p, Capacitor_SMD:C_0805_2012Metric, symbol Device:C
- removed D1: D_Schottky, PMEG4010BEA:SOD323F_NEX, symbol Device:D_Schottky
- removed D3, D4, D5, D6: 1N4002, Diode_THT:D_DO-41_SOD81_P10.16mm_Horizontal, symbol Diode:1N4002
- removed J1: DeployLipo, TerminalBlock_Phoenix:TerminalBlock_Phoenix_MKDS-3-2-5.08_1x02_P5.08mm_Horizontal, symbol Connector:Conn_01x02_Male
- removed J2: Conn_01x04, Connector_PinHeader_2.54mm:PinHeader_1x04_P2.54mm_Vertical, symbol Connector_Generic:Conn_01x04
- removed J9: UCLipo, Connector_JST:JST_PH_B2B-PH-K_1x02_P2.00mm_Vertical, symbol Connector:Conn_01x02_Male
- removed R1: 162k, Resistor_SMD:R_0402_1005Metric, symbol Device:R
- removed R2: 10k, Resistor_SMD:R_0402_1005Metric, symbol Device:R
- removed R3, R6: 240, Resistor_SMD:R_0402_1005Metric, symbol Device:R
- removed R5: 4.56k, Resistor_SMD:R_0402_1005Metric, symbol Device:R
- removed R7: 720, Resistor_SMD:R_0402_1005Metric, symbol Device:R
- removed U3: LM317LCLPRE3, LM317MDT_TR:DPAK_STM, symbol LM317MDT_TR:LM317MDT-TR
- added C1, C3: 4.7uF 50V, Capacitor_SMD:C_0603_1608Metric, symbol Device:C_Small
- added C10, C9: 10uF, Capacitor_SMD:C_0805_2012Metric, symbol Device:C_Small
- added C11: 620pF, Capacitor_SMD:C_0402_1005Metric, symbol Device:C_Small
- added C2, C8: 4.7uF, Capacitor_SMD:C_0603_1608Metric, symbol Device:C_Small
- added C4: 4.7pF 50V, Capacitor_SMD:C_0402_1005Metric, symbol Device:C_Small
- added C5: 100nF 50V, Capacitor_SMD:C_0402_1005Metric, symbol Device:C_Small
- added C6: 1uF 50V, Capacitor_SMD:C_0603_1608Metric, symbol Device:C_Small
- added C7: 1uF, Capacitor_SMD:C_0603_1608Metric, symbol Device:C_Small
- added D1: PMEG6010CEJ, Diode_SMD:D_SOD-323F, symbol Diode:PMEG6010CEJ
- added J1: Conn_01x02_Pin, Connector_Molex:Molex_Nano-Fit_105313-xx02_1x02_P2.50mm_Horizontal, symbol Connector:Conn_01x02_Pin
- added J2: DeployLipo, Connector_AMASS:AMASS_XT60PW-M_1x02_P7.20mm_Horizontal, symbol Connector:Conn_01x02_Male
- added J3: Conn_01x03_Pin, Connector_Molex:Molex_Nano-Fit_105313-xx03_1x03_P2.50mm_Horizontal, symbol Connector:Conn_01x03_Pin
- added L2: 2.2uH, Inductor_SMD:L_0805_2012Metric, symbol Device:L_Small
- added R1: 162k, Resistor_SMD:R_0402_1005Metric, symbol Device:R_Small
- added R2: 240Ω, Resistor_SMD:R_0402_1005Metric, symbol Device:R_Small
- added R3: 4.56kΩ, Resistor_SMD:R_0402_1005Metric, symbol Device:R_Small
- added R4: 10k, Resistor_SMD:R_0402_1005Metric, symbol Device:R_Small
- added R5: 100k, Resistor_SMD:R_0402_1005Metric, symbol Device:R_Small
- added R6: 953k, Resistor_SMD:R_0402_1005Metric, symbol Device:R_Small
- added R7: 180k, Resistor_SMD:R_0402_1005Metric, symbol Device:R_Small
- added U4: TPS62150, Package_DFN_QFN:VQFN-16-1EP_3x3mm_P0.5mm_EP1.68x1.68mm_ThermalVias, symbol Regulator_Switching:TPS62150
- L1: value 8.2u -> 6.8uH; footprint CDR7D28MNNP-8R0NC:IND_8R0NC_SUM -> iclr:WE-HEPC_6030; MPN (none) -> 78408063006
- U2: renamed from U4; value LM317LCLPRE3 -> LM317LIDR; footprint LM317MDT_TR:DPAK_STM -> iclr:SOIC127P599X175-8N
- renumbered H101 to H1, H102 to H2, H103 to H3, H104 to H4, U2 to U1, U1 to U3
Connections:
- net BBIN: now also U3.4 (EN/UVLO), C2.1, C8.1, U4.10 (VIN), U4.11 (VIN), U4.12 (VIN), U4.13 (EN)
- net Filtered_Power_Out_25V: now also U2.2 (VOUT), U2.6 (VOUT), U2.7 (VOUT), C6.1, J3.3 (Pin_3), R2.1
- net GND: now also U1.4 (GND), U1.7 (GND), C1.2, C10.2, C11.2, C2.2, C3.2, C5.2, C6.2, C7.2, C8.2, C9.2, J1.1 (Pin_1), J2.1 (Pin_1), J3.1 (Pin_1), R3.2, R4.2, R7.2, U4.15 (GND), U4.16 (GND), U4.17 (GND), U4.6 (GND), U4.8 (DEF)
- net ON-OFF: now also J1.2 (Pin_2)
- net Power_Out_27.5V: now also U2.1 (VIN), C3.1, C4.1, C5.1, D1.1 (K), R1.1; no longer U2.2 (VIN)
- net Power_Out_5V: now also C10.1, C9.1, J3.2 (Pin_2), L2.2, R5.1, R6.1, U4.14 (VOS), U4.7 (FSW)
- net at U3.3 (FBX): now also C4.2, R1.2, R4.1
- net at L1.2, U3.1 (SW): now also D1.2 (A)
- net BATT+: now reaches U1.6 (VIN)
- net BATT+: now also C1.1, J2.2 (Pin_2)
- net at U3.5 (INTVCC): now also C7.1; no longer U3.4 (EN/UVLO)
- new net: R6.2, R7.1, U4.5 (FB)
- new net: R2.2, R3.1, U2.4 (ADJUST)
- new net: U2.5 (NC), U2.8 (NC)
- new net: L2.1, U4.1 (SW), U4.2 (SW), U4.3 (SW)
- new net: R5.2, U4.4 (PG)
- new net: C11.1, U4.9 (SS/TR)
- no-connect marks 0 -> 1
Other:
- note added: "https://webench.ti.com/appinfo/webench/scripts/SDP.cgi?ID=9BC53E732B25D161"
- note added: "need min 5mA to maintain regulation so R is low"
- moved on the sheet: H1, H2, H3, H4, L1, U1, U3

Commit message: updated detector - need to order
Parts:
- R1: value 162k -> 162kΩ
- R4: value 10k -> 10kΩ
- R5: value 100k -> 100kΩ
- R6: value 953k -> 953kΩ
- R7: value 180k -> 180kΩ
Connections:
- net GND: now also J3.2 (Pin_2); no longer J3.1 (Pin_1)
- net Power_Out_5V: now also J3.1 (Pin_1); no longer J3.2 (Pin_2)
Other:
- moved on the sheet: C10, C9, R6, R7

Commit message: new docs/3d files
Parts:
- J1, J2, J3: now not fitted
- R3: value 4.56kΩ -> 4.53kΩ
Changed lines of the file:
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@@
 	(text "need min 5mA to maintain regulation so R is low"
 		(exclude_from_sim no)
-		(at 230.886 114.808 0)
+		(at 247.142 114.3 0)
 		(effects
 			(font
@@
 			)
 		)
-		(property "Value" "4.56kΩ"
+		(property "Value" "4.53kΩ"
 			(at 228.346 107.95 0)
 			(show_name no)
@@
 		(on_board yes)
 		(in_pos_files yes)
-		(dnp no)
+		(dnp yes)
 		(property "Reference" "J2"
 			(at 62.865 52.07 0)
@@
 		(on_board yes)
 		(in_pos_files yes)
-		(dnp no)
+		(dnp yes)
 		(property "Reference" "J3"
 			(at 167.64 35.56 0)
@@
 		(on_board yes)
 		(in_pos_files yes)
-		(dnp no)
+		(dnp yes)
 		(property "Reference" "J1"
 			(at 67.31 26.162 0)
