File: raven-main/Detector-Proto-Board/Detector-Proto-Board.kicad_sch (KiCad schematic)
At the start: 40 parts, among them IC1 ADA4817-1ARDZ-R7, J1 Conn_01x04, J2 Conn_01x01, J3 Conn_01x02, U9 TLV3201AIDCKT

Commit message: power board done
Parts:
- removed J1: Conn_01x04, Connector_PinHeader_2.54mm:PinHeader_1x04_P2.54mm_Vertical, symbol Connector_Generic:Conn_01x04
- removed J3: Conn_01x02, Connector_PinHeader_2.54mm:PinHeader_1x02_P2.54mm_Vertical, symbol Connector_Generic:Conn_01x02
- added J3: Conn_01x02_Pin, Connector_Molex:Molex_Nano-Fit_105313-xx02_1x02_P2.50mm_Horizontal, symbol Connector:Conn_01x02_Pin
- added J4: Conn_01x03_Pin, Connector_Molex:Molex_Nano-Fit_105313-xx03_1x03_P2.50mm_Horizontal, symbol Connector:Conn_01x03_Pin
- added TP6, TP7: TestPoint, symbol Connector:TestPoint
Connections:
- net +5V: now also J4.3 (Pin_3)
- net GND: now also J3.2 (Pin_2), J4.2 (Pin_2)
- net at C35.1, C42.1, D4.2 (A)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: now also TP7.1
- net at C39.1, D4.1 (K), D5.1 (K)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: now also TP6.1
- net at D1.2 (A2): now also J4.1 (Pin_1)
- net Detector_Out_A renamed Detector_Out
- net Detector_Out: now also J3.1 (Pin_1)
- net V_thresh_A renamed V_thresh
Other:
- moved on the sheet: D2, D4, D5, H101, H102, H103, H104, R30, TP5

Commit message: updated detector - need to order
Parts:
- removed C1: 330p, Capacitor_SMD:C_0402_1005Metric, symbol Device:C
- removed C35, C42: 0.5pF, Capacitor_SMD:C_0402_1005Metric, symbol Device:C
- removed C36: 10uF, Capacitor_SMD:C_0402_1005Metric, symbol Device:C
- removed C37, C38, C39: 100nF, Capacitor_SMD:C_0402_1005Metric, symbol Device:C
- removed C40: 1uF, Capacitor_SMD:C_0402_1005Metric, symbol Device:C
- removed D1: SMAJ26A, Diode_SMD:D_SMA, symbol Diode:SMAJ26A
- removed R1, R38: 0, Resistor_SMD:R_0402_1005Metric, symbol Device:R
- removed R2: 1k, Resistor_SMD:R_0402_1005Metric, symbol Device:R
- removed R27, R37: 1G, Resistor_SMD:R_0402_1005Metric, symbol Device:R
- removed R29: R_Variable, 3224X:SOT_502E, symbol Device:R_Variable
- removed R3: 2k, Resistor_SMD:R_0402_1005Metric, symbol Device:R
- removed R30: 10K, Resistor_SMD:R_0402_1005Metric, symbol Device:R
- removed R31: 390K, Resistor_SMD:R_0402_1005Metric, symbol Device:R
- removed R32: 33, Resistor_SMD:R_0402_1005Metric, symbol Device:R_Small
- removed R33, R34: 10k, Resistor_SMD:R_0402_1005Metric, symbol Device:R
- removed R35: 1.6k, Resistor_SMD:R_0402_1005Metric, symbol Device:R
- removed TP1: OUT, TestPoint:TestPoint_Pad_D2.5mm, symbol Connector:TestPoint
- removed TP4: Detector_Out, TestPoint:TestPoint_Pad_D2.5mm, symbol Connector:TestPoint
- removed TP7: TestPoint, symbol Connector:TestPoint
- added C1: 100nF 50V, Capacitor_SMD:C_0402_1005Metric, symbol Device:C_Small
- added C2: 1uF, Capacitor_SMD:C_0603_1608Metric, symbol Device:C_Small
- added C3: 1pF, Capacitor_SMD:C_0402_1005Metric, symbol Device:C_Small
- added C4, C7: 100nF, Capacitor_SMD:C_0402_1005Metric, symbol Device:C_Small
- added C5: 10uF, Capacitor_SMD:C_0805_2012Metric, symbol Device:C_Small
- added C6: 330pF, Capacitor_SMD:C_0402_1005Metric, symbol Device:C_Small
- added R1, R2, R4: 10kΩ, Resistor_SMD:R_0402_1005Metric, symbol Device:R_Small
- added R10, R3: 0Ω, Resistor_SMD:R_0402_1005Metric, symbol Device:R_Small
- added R11: 1.6kΩ, Resistor_SMD:R_0402_1005Metric, symbol Device:R_Small
- added R12: 390kΩ, Resistor_SMD:R_0402_1005Metric, symbol Device:R_Small
- added R13: 1kΩ, Resistor_SMD:R_0402_1005Metric, symbol Device:R_Small
- added R14: 2kΩ, Resistor_SMD:R_0402_1005Metric, symbol Device:R_Small
- added R5, R6: 1GΩ, Resistor_SMD:R_0402_1005Metric, symbol Device:R_Small
- added R7: 33Ω, Resistor_SMD:R_0402_1005Metric, symbol Device:R_Small
- added RV1: 3214W-1-102E, Potentiometer_SMD:Potentiometer_Bourns_3214W_Vertical, symbol Device:R_Potentiometer
- added TP2: 25V, TestPoint:TestPoint_Pad_D2.0mm, symbol Connector:TestPoint
- R9: renamed from R28; value 100k -> 100kΩ
- TP1: renamed from TP3; footprint TestPoint:TestPoint_Pad_D2.5mm -> TestPoint:TestPoint_Pad_D2.0mm
- TP3: renamed from TP2; footprint TestPoint:TestPoint_Pad_D2.5mm -> TestPoint:TestPoint_Pad_D2.0mm
- TP5: value GND -> OUT; footprint TestPoint:TestPoint_Pad_D2.5mm -> TestPoint:TestPoint_Pad_D2.0mm
- TP6: value TestPoint -> Detector_Out; footprint (none) -> TestPoint:TestPoint_Pad_D2.0mm
- renumbered D4 to D1, D5 to D2, D2 to D3, H101 to H1, H102 to H2, H103 to H3, H104 to H4, J4 to J1, U9 to U1
Connections:
- net +25V: now also J1.1 (Pin_1), R1.1
- net +5V: now also C4.1, C5.1, C7.1, R2.1
- net Detector_Out: now also TP6.1, R13.2, R14.1
- net GND: now also C1.2, C2.2, C4.2, C5.2, C6.2, C7.2, R14.2, R4.2; no longer TP5.1
- net OUT: now also TP5.1, C3.1, R11.2, R5.1, R6.1
- net V_thresh: now also R10.2, R12.2
- net Vped: now also C2.1, R3.2, R4.1, R7.1
- net at D1.1 (K), D2.1 (K): now also C1.1, R1.2, TP2.1; no longer TP6.1
- net at U1.4 (IN-): now also C6.1, R11.1
- net at D1.2 (A), D2.2 (A), IC1.2 (-IN): now also C3.2, R5.2, R6.2
- net at R9.1: now also R10.1, RV1.3
- net Detector_Out_5V: now reaches U1.1 (OUT)
- net Detector_Out_5V: now also R12.1, R13.1
- new net: R7.2, RV1.2
- new net: R2.2, R3.1
- no-connect marks 1 -> 2
Other:
- note added: "Charge Amplifier"
- note added: "Input Connector"
- note added: "Photodiodes"
- note added: "Processing Inputs"
- note removed: "Clean up supply to Op-Amp"
- moved on the sheet: D1, D2, D3, IC1, J1, J2, J3, R9, TP1, TP3, U1

Commit message: new docs/3d files
Parts:
- removed R5: 1GΩ, Resistor_SMD:R_0402_1005Metric, symbol Device:R_Small
- added C4: 1uF 50V, Capacitor_SMD:C_0603_1608Metric, symbol Device:C_Small
- D3: value SMAJ5.0A -> SMAJ6.0A
- J1, J2, J3: now not fitted
- R5: renamed from R6; value 1GΩ -> 470MΩ; footprint Resistor_SMD:R_0402_1005Metric -> Resistor_SMD:R_0603_1608Metric
- TP1, TP2, TP3: now left out of the parts list
- TP4: renamed from TP5; now left out of the parts list
- TP5: renamed from TP6; now left out of the parts list
- renumbered C4 to C5, C5 to C6, C6 to C7, C7 to C8, R12 to R10, R13 to R11, R14 to R12, R7 to R6, R9 to R7, R10 to R8, R11 to R9
Connections:
- net +25V: now also C4.1
- net GND: now also C4.2
